File: Hardware/MultiBASIC040.kicad_sch (KiCad schematic)
At the start: 20 parts, among them J8 HDDLED, J8 PWRLED, U1 MC68LC040

Commit message: DRC cleanup
Parts:
- removed J8: PWRLED, Connector_PinHeader_2.54mm:PinHeader_1x02_P2.54mm_Vertical, symbol Connector_Generic:Conn_01x02
- removed J8: HDDLED, Connector_PinHeader_2.54mm:PinHeader_1x02_P2.54mm_Vertical, symbol Connector_Generic:Conn_01x02
- removed R10, R56: 1k, Resistor_SMD:R_0402_1005Metric, symbol Device:R_Small
Other:
- sheet Bus Control ports: added none; removed IDE-DASP
